File: NitrogenGenerator.kicad_pcb (KiCad board)
At the start: 2 copper layers, 147 x 55 mm, 21 parts, among them J1 Conn_ARM_SWD_TagConnect_TC203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, J2 Screw_Terminal_01x10, K1 AA28F-R1, K2 AA28F-R1, U1 STM32G030F6Px, U2 IRM-45-24, U3 R-78E5.0-0.5, U4 TLV70433DBVR

Commit message: .
Parts:
- added D1: 1N4007, Diode_SMD:D_SOD-123F, F.Cu at (142.6, 67.8)
- added D2: 1N4007, Diode_SMD:D_SOD-123F, F.Cu at (142.6, 57.4)
- added J3: ERM19264-4, NitrogenGenerator:ERM19264DNS-4, B.Cu at (140.3, 34.8)
- added J4: 726386-2, NitrogenGenerator:CONN_726386-2_TEC, F.Cu at (23.0, 56.5)
- added J5: 726386-2, NitrogenGenerator:CONN_726386-2_TEC, F.Cu at (22.9, 41.9)
- moved R6 4.55 mm to (124.0, 28.0)
- moved R3 4.55 mm to (125.8, 28.0)
- moved R4 4.55 mm to (125.8, 24.9)
- moved R5 4.55 mm to (124.0, 24.9)
- moved J2 1.96 mm to (146.8, 69.8)
Connections:
- R3 pad 1: /CTRL_VALVE_IN -> /PRESSURE_INPUT
- R4 pad 1: /CTRL_VALVE_OUT -> /PRESSURE_OUTPUT
- R5 pad 2: /CTRL_VALVE_OUT -> /PRESSURE_OUTPUT
- R6 pad 2: /CTRL_VALVE_IN -> /PRESSURE_INPUT
- U1 pad 1: unconnected-(U1-PB7/PB8-Pad1) -> GND
- U1 pad 15: unconnected-(U1-PA8/PB0/PB1/PB2-Pad15) -> GND
- U1 pad 16: unconnected-(U1-PA9/PA11-Pad16) -> GND
- U1 pad 17: unconnected-(U1-PA10/PA12-Pad17) -> GND
- U1 pad 2: unconnected-(U1-PB9/PC14-Pad2) -> GND
- U1 pad 20: unconnected-(U1-PB3/PB4/PB5/PB6-Pad20) -> GND
- U1 pad 3: unconnected-(U1-PC15-Pad3) -> GND
- U1 pad 9: unconnected-(U1-PA2-Pad9) -> GND
- U2 pad 1: unconnected-(U2-AC/L-Pad1) -> Net-(U2-AC/L)
- U2 pad 2: unconnected-(U2-AC/N-Pad2) -> Net-(U2-AC/N)
Routing:
- net +3.3V: track 33.7 -> 68.9 mm, vias 2 -> 3
- net Net-(U2-AC/N): track 0.00 -> 30.3 mm
- net /LCD_CD: track 0.00 -> 28.1 mm, vias 0 -> 1
- net /LCD_SCK: track 0.00 -> 27.0 mm, vias 0 -> 1
- net /LCD_SDA: track 0.00 -> 26.1 mm, vias 0 -> 1
- net Net-(U2-AC/L): track 0.00 -> 20.4 mm
- net Net-(J2-Pin_7): track 20.8 -> 38.1 mm
- net +24V: track 63.2 -> 76.8 mm
- net /PRESSURE_OUTPUT: track 0.00 -> 9.58 mm
- net Net-(J2-Pin_10): track 18.1 -> 24.2 mm
- net /LOAD_VALVE_IN: track 16.4 -> 21.3 mm
- net /CTRL_VALVE_OUT: track 34.0 -> 29.2 mm, vias 2 -> 0
- net /LOAD_VALVE_OUT: track 16.3 -> 20.4 mm
- net /PRESSURE_INPUT: track 0.00 -> 3.38 mm
- net GND: track 3.11 -> 6.19 mm, vias 6 -> 10
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Other:
- board size 147 x 55 mm -> 155 x 55 mm
- board text added: "24V"
- board text added: "5V"
- board text added: "GND"
- board text added: "NITROGEN GENERATOR CONTROLLER"
- board text added: "SNS1"
- board text added: "SNS2"
- board text added: "VLV1"
- board text added: "VLV2"

Commit message: .
Parts:
- moved J2 5.40 mm to (152.2, 69.8)
Routing:
- net +24V: track 76.8 -> 93.0 mm
- net Net-(J2-Pin_7): track 38.1 -> 43.5 mm
- net Net-(J2-Pin_10): track 24.2 -> 29.6 mm
- net +5V: track 68.8 -> 74.2 mm
- net /LOAD_VALVE_OUT: track 20.4 -> 25.8 mm
- net /LOAD_VALVE_IN: track 21.3 -> 26.7 mm
- net GND: vias 10 -> 6
- net (no net): vias 0 -> 4
Other:
- board size 155 x 55 mm -> 160 x 55 mm

Commit message: .
Parts:
- added J6: Conn_01x06_Pin, Connector_PinHeader_2.54mm:PinHeader_1x06_P2.54mm_Vertical, F.Cu at (146.5, 28.0)
Connections:
- J1 pad 6: /SWO -> unconnected-(J1-SWO-Pad6)
- U1 pad 1: GND -> unconnected-(U1-PB7/PB8-Pad1)
- U1 pad 13: /LCD_SDA -> /LCD_CD
- U1 pad 14: /LCD_CD -> /LCD_SDA
- U1 pad 20: GND -> /UART1_TX
Routing:
- net /UART1_TX: track 0.00 -> 67.4 mm, vias 0 -> 1
- net /SWDIO: track 10.5 -> 63.8 mm, vias 0 -> 1
- net /SWCLK: track 13.2 -> 60.2 mm, vias 0 -> 1
- net /~{RESET}: track 10.4 -> 46.6 mm
- net +3.3V: track 68.9 -> 75.0 mm
Other:
- board text added: "3.3V"
- board text added: "NRST"
- board text added: "SWCK"
- board text added: "SWDA"
- board text added: "UART"

Commit message: .
Parts:
- moved J3 4.60 mm to (135.7, 34.9)
- moved J6 1.59 mm to (145.0, 28.3)
Connections:
- J1 pad 6: unconnected-(J1-SWO-Pad6) -> /UART1_TX
Routing:
- net /UART1_TX: track 67.4 -> 72.9 mm
- net /LCD_CD: track 28.4 -> 23.3 mm
- net /LCD_SCK: track 27.0 -> 22.3 mm
- net /LCD_SDA: track 26.3 -> 21.7 mm
- net +3.3V: track 75.0 -> 71.7 mm
- net /SWCLK: track 60.2 -> 60.7 mm
- net Net-(J2-Pin_7): track 43.5 -> 43.0 mm
- net GND: vias 6 -> 38
Other:
- board text added: "+24V"
- board text added: "+5V"
- board text added: "BY TINIC"
- board text added: "L"
- board text added: "N"
- board text added: "NITROGEN GENERATOR V1.5 2025"
- board text added: "SENSE1"
- board text added: "SENSE2"
- board text added: "VALVE1"
- board text added: "VALVE2"
- board text removed: "24V"
- board text removed: "5V"
- board text removed: "NITROGEN GENERATOR CONTROLLER"
- board text removed: "SNS1"
- board text removed: "SNS2"
- board text removed: "VLV1"
- board text removed: "VLV2"
