File: NitrogenGenerator.kicad_pcb (KiCad board)
At the start: 2 copper layers, 160 x 55 mm, 27 parts, among them J1 Conn_ARM_SWD_TagConnect_TC203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, J2 Screw_Terminal_01x10, J3 ERM19264-4, J4 726386-2, J5 726386-2, J6 Conn_01x06_Pin, K1 AA28F-R1, K2 AA28F-R1, U1 STM32G030F6Px, U2 IRM-45-24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

Commit message: .
Connections:
- J3 pad 7: +3.3V -> /LCD_RESET
- J3 pad 9: GND -> /LCD_CS
- U1 pad 15: GND -> /LCD_CS
- U1 pad 16: GND -> /LCD_RESET
Routing:
- net /LCD_RESET: track 0.00 -> 34.9 mm, vias 0 -> 1
- net /LCD_CS: track 0.00 -> 24.3 mm, vias 0 -> 1
- net +3.3V: track 71.7 -> 60.1 mm
- net GND: track 6.19 -> 14.3 mm, vias 38 -> 37

Commit message: .
Other:
- board text added: "BY TINIC 2025-04-21"
- board text added: "NITROGEN GENERATOR V1.6 #146"
- board text removed: "BY TINIC"
- board text removed: "NITROGEN GENERATOR V1.5 2025"
Changed lines of the file:
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@@
 		(layer "Edge.Cuts")
 	)
-	(gr_text "BY TINIC"
+	(gr_text "BY TINIC 2025-04-21"
 		(at 176.66 64.55 90)
 		(layer "F.SilkS")
@@
 		)
 	)
-	(gr_text "NITROGEN GENERATOR V1.5 2025"
+	(gr_text "NITROGEN GENERATOR V1.6 #146"
 		(at 174.49 64.6 90)
 		(layer "F.SilkS")
