File: NitrogenGenerator.kicad_pcb (KiCad board)
At the start: 2 copper layers, 160 x 55 mm, 29 parts, among them J1 Conn_ARM_SWD_TagConnect_TC203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, J2 Screw_Terminal_01x10, J3 ERM19264-4, J4 726386-2, J5 726386-2, J6 Conn_01x06_Pin, K1 AA28F-R1, K2 AA28F-R1, U1 STM32G030F6Px, U2 IRM-45-24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

Commit message: .
Parts:
- added R7: 100, Resistor_SMD:R_0603_1608Metric, F.Cu at (130.9, 28.1)
Connections:
- J3 pad 2: +3.3V -> Net-(J3-Pin_2)
Routing:
- net +5V: track 74.2 -> 95.4 mm, vias 1 -> 2
- net Net-(J3-Pin_2): track 0.00 -> 5.53 mm
- net +3.3V: track 60.1 -> 55.2 mm
