File: NitrogenGenerator.kicad_sch (KiCad schematic)
At the start: 3 parts, among them K1 AA28F-R1, K2 AA28F-R1, U1 STM32G030F6Px

Commit message: .
Parts:
- added C1, C2, C3: 0.1uF, Capacitor_SMD:C_0603_1608Metric, symbol Device:C
- added C4, C5, C6, C7: 4.7uF, Capacitor_SMD:C_0603_1608Metric, symbol Device:C
- added J1: Conn_ARM_SWD_TagConnect_TC2030-NL, Connector:Tag-Connect_TC2030-IDC-NL_2x03_P1.27mm_Vertical, symbol Connector:Conn_ARM_SWD_TagConnect_TC2030-NL
- added J2: Screw_Terminal_01x10, TerminalBlock_RND:TerminalBlock_RND_205-00284_1x10_P5.00mm_Vertical, symbol Connector:Screw_Terminal_01x10
- added J3: ERM19264-4, Display:ERM19264, symbol Connector:Conn_01x09_Pin
- added R1, R2: 1.6K, Resistor_SMD:R_0603_1608Metric, symbol Device:R
- added R3, R4: 10K, Resistor_SMD:R_0603_1608Metric, symbol Device:R
- added R5, R6: 20K, Resistor_SMD:R_0603_1608Metric, symbol Device:R
- added U2: IRM-45-24, NitrogenGenerator:IRM-45_MWU, symbol NitrogenGenerator:IRM-45-12
- added U3: R-78E5.0-0.5, NitrogenGenerator:R-78E-0.5_RCP, symbol NitrogenGenerator:R-78E5.0-0.5
- added U4: TLV70433DBVR, NitrogenGenerator:TLV70433DBVR, symbol NitrogenGenerator:TLV70433DBVR
- K1, K2: footprint SMD6_AA28F-R1_BTI -> NitrogenGenerator:SMD6_AA28F-R1_BTI
Connections:
- net CTRL_VALVE_OUT: now reaches K2.1
- net CTRL_VALVE_OUT: now also U1.8 (PA1), R4.1, R5.2
- net at K2.2: now also R2.2
- net LOAD_VALVE_OUT: now reaches K2.4
- net LOAD_VALVE_OUT: now also K2.6, J2.3 (Pin_3)
- net GND: now reaches K2.5
- net GND: now also K1.5, U1.5 (VSS), C1.2, C2.2, C3.2, C4.2, C5.2, C6.2, C7.2, J1.5 (GND), J2.6 (Pin_6), J2.9 (Pin_9), J3.3 (Pin_3), J3.9 (Pin_9), R1.1, R2.1, R5.1, R6.1, U2.4 (V-), U3.2 (GND), U4.1 (GND)
- net CTRL_VALVE_IN: now reaches K1.1
- net CTRL_VALVE_IN: now also U1.7 (PA0), R3.1, R6.2
- net at K1.2: now also R1.2
- net LOAD_VALVE_IN: now reaches K1.4
- net LOAD_VALVE_IN: now also K1.6, J2.1 (Pin_1)
- net PRESSURE_INPUT: now reaches U1.10 (PA3)
- net PRESSURE_OUTPUT: now reaches U1.11 (PA4)
- net LCD_SCK: now reaches U1.12 (PA5)
- net LCD_SCK: now also J3.5 (Pin_5)
- net LCD_SDA: now reaches U1.13 (PA6)
- net LCD_SDA: now also J3.6 (Pin_6)
- net LCD_CD: now reaches U1.14 (PA7)
- net LCD_CD: now also J3.8 (Pin_8)
- net SWDIO: now reaches U1.18 (PA13)
- net SWDIO: now also J1.2 (SWDIO)
- net SWCLK: now reaches U1.19 (PA14/PA15)
- net SWCLK: now also J1.4 (SWCLK)
- net +3.3V: now reaches U1.4 (VDD)
- net +3.3V: now also C1.1, C2.1, C7.1, J1.1 (VCC), U4.3 (OUT)
- net ~{RESET}: now reaches U1.6 (NRST)
- net ~{RESET}: now also J1.3 (~{RESET})
- new net: J2.10 (Pin_10), R4.2
- new net: J2.7 (Pin_7), R3.2
- new net +24V: C5.1, C6.1, J2.2 (Pin_2), J2.4 (Pin_4), U2.3 (V+), U3.1 (+VIN)
- new net +5V: C3.1, C4.1, J2.5 (Pin_5), J2.8 (Pin_8), J3.4 (Pin_4), J3.7 (Pin_7), U3.3 (+VOUT), U4.2 (IN)
- new net SWO: J1.6 (SWO)
- no-connect marks 0 -> 12
Other:
- moved on the sheet: K1, K2, U1

Commit message: .
Connections:
- net +3.3V: now also J3.2 (Pin_2), J3.4 (Pin_4), J3.7 (Pin_7)
- net +5V: no longer J3.4 (Pin_4), J3.7 (Pin_7)
- net GND: now also J3.1 (Pin_1)
- no-connect marks 12 -> 10
Changed lines of the file:
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@@
+	)
+	(junction
+		(at 97.79 101.6)
+		(diameter 0)
+		(color 0 0 0 0)
 	)
 	(junction
@@
 	)
 	(junction
+		(at 93.98 99.06)
+		(diameter 0)
+		(color 0 0 0 0)
+	)
+	(junction
 		(at 88.9 163.83)
 		(diameter 0)
@@
 	)
 	(no_connect
-		(at 101.6 96.52)
-	)
-	(no_connect
 		(at 99.06 48.26)
 	)
@@
 		(at 149.86 60.96)
 	)
-	(no_connect
-		(at 101.6 99.06)
-	)
 	(wire
 		(pts
@@
 	(wire
 		(pts
+			(xy 93.98 99.06) (xy 101.6 99.06)
+		)
+		(stroke
+			(width 0)
+			(type default)
+		)
+	)
+	(wire
+		(pts
 			(xy 210.82 140.97) (xy 210.82 143.51)
 		)
@@
 	(wire
 		(pts
+			(xy 101.6 96.52) (xy 97.79 96.52)
+		)
+		(stroke
+			(width 0)
+			(type default)
+		)
+	)
+	(wire
+		(pts
 			(xy 195.58 54.61) (xy 214.63 54.61)
 		)
@@
 	(wire
 		(pts
-			(xy 93.98 93.98) (xy 93.98 104.14)
+			(xy 93.98 93.98) (xy 93.98 99.06)
 		)
 		(stroke
@@
 		(pts
 			(xy 195.58 31.75) (xy 195.58 39.37)
+		)
+		(stroke
+			(width 0)
+			(type default)
+		)
+	)
+	(wire
+		(pts
+			(xy 97.79 96.52) (xy 97.79 101.6)
+		)
+		(stroke
+			(width 0)
+			(type default)
+		)
+	)
+	(wire
+		(pts
+			(xy 93.98 99.06) (xy 93.98 104.14)
 		)
 		(stroke
@@
 			)
 		)
-		(property "Value" "+5V"
+		(property "Value" "+3.3V"
 			(at 93.98 88.9 0)
 			(effects

Commit message: .
Parts:
- added D1, D2: 1N4007, Diode_SMD:D_SOD-123F, symbol Diode:1N4007
- added J4, J5: 726386-2, NitrogenGenerator:CONN_726386-2_TEC, symbol NitrogenGenerator:726386-2
- J3: footprint Display:ERM19264 -> NitrogenGenerator:ERM19264DNS-4
Connections:
- net +24V: now also D1.1 (K), D2.1 (K)
- net CTRL_VALVE_IN: no longer R3.1, R6.2
- net CTRL_VALVE_OUT: no longer R4.1, R5.2
- net GND: now also U1.1 (PB7/PB8), U1.15 (PA8/PB0/PB1/PB2), U1.16 (PA9/PA11), U1.17 (PA10/PA12), U1.2 (PB9/PC14), U1.20 (PB3/PB4/PB5/PB6), U1.3 (PC15), U1.9 (PA2)
- net LOAD_VALVE_IN: now also D1.2 (A)
- net LOAD_VALVE_OUT: now also D2.2 (A)
- net PRESSURE_INPUT: now also R3.1, R6.2
- net PRESSURE_OUTPUT: now also R4.1, R5.2
- net at U2.1 (AC/L): now also J5.1, J5.2
- net at U2.2 (AC/N): now also J4.1, J4.2
- no-connect marks 10 -> 2
Other:
- moved on the sheet: U1

Commit message: .
Parts:
- added J6: Conn_01x06_Pin, Connector_PinHeader_2.54mm:PinHeader_1x06_P2.54mm_Vertical, symbol Connector:Conn_01x06_Pin
Connections:
- net +3.3V: now also J6.1 (Pin_1)
- net GND: now also J6.6 (Pin_6); no longer U1.1 (PB7/PB8), U1.20 (PB3/PB4/PB5/PB6)
- net LCD_CD: now also U1.13 (PA6); no longer U1.14 (PA7)
- net LCD_SDA: now also U1.14 (PA7); no longer U1.13 (PA6)
- net SWCLK: now also J6.3 (Pin_3)
- net SWDIO: now also J6.4 (Pin_4)
- net ~{RESET}: now also J6.2 (Pin_2)
- net SWO: no longer names the net of J1.6 (SWO)
- new net UART1_TX: J6.5 (Pin_5), U1.20 (PB3/PB4/PB5/PB6)
- no-connect marks 2 -> 4
Other:
- moved on the sheet: C1, C2, C3, C4, C5, C6, C7, J2, R3, R4, R5, R6

Commit message: .
Connections:
- net UART1_TX: now also J1.6 (SWO)
- no-connect marks 4 -> 3
Changed lines of the file:
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@@
-	)
-	(no_connect
-		(at 41.91 167.64)
 	)
 	(no_connect
@@
 	(wire
 		(pts
+			(xy 41.91 167.64) (xy 52.07 167.64)
+		)
+		(stroke
+			(width 0)
+			(type default)
+		)
+	)
+	(wire
+		(pts
 			(xy 133.35 154.94) (xy 142.24 154.94)
 		)
@@
 		)
 	)
+	(label "UART1_TX"
+		(at 52.07 167.64 180)
+		(effects
+			(font
+				(size 1.27 1.27)
+			)
+			(justify right bottom)
+		)
+	)

Commit message: .
Other:
- added sheet PnID (PnID.kicad_sch)
Changed lines of the file:
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@@
+		)
+	)
+	(sheet
+		(at 236.22 140.97)
+		(size 41.91 19.05)
+		(exclude_from_sim no)
+		(in_bom yes)
+		(on_board yes)
+		(dnp no)
+		(fields_autoplaced yes)
+		(stroke
+			(width 0.1524)
+			(type solid)
+		)
+		(fill
+			(color 0 194 194 1.0000)
+		)
+		(property "Sheetname" "PnID"
+			(at 236.22 140.2584 0)
+			(effects
+				(font
+					(size 1.27 1.27)
+				)
+				(justify left bottom)
+			)
+		)
+		(property "Sheetfile" "PnID.kicad_sch"
+			(at 236.22 160.6046 0)
+			(effects
+				(font
+					(size 1.27 1.27)
+				)
+				(justify left top)
+			)
+		)
+		(instances
+			(project "NitrogenGenerator"
+				(path "/c5365556-9b4a-4e37-8bb8-20fd18113201"
+					(page "2")
+				)
+			)
 		)
 	)

Commit message: .
Connections:
- net +3.3V: no longer J3.7 (Pin_7)
- net GND: no longer J3.9 (Pin_9), U1.15 (PA8/PB0/PB1/PB2), U1.16 (PA9/PA11)
- new net LCD_CS: J3.9 (Pin_9), U1.15 (PA8/PB0/PB1/PB2)
- new net LCD_RESET: J3.7 (Pin_7), U1.16 (PA9/PA11)
Changed lines of the file:
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@@
-	)
-	(junction
-		(at 93.98 104.14)
-		(diameter 0)
-		(color 0 0 0 0)
 	)
 	(junction
@@
 	)
 	(junction
-		(at 160.02 59.69)
-		(diameter 0)
-		(color 0 0 0 0)
-	)
-	(junction
 		(at 133.35 154.94)
 		(diameter 0)
@@
 	)
 	(junction
-		(at 97.79 116.84)
-		(diameter 0)
-		(color 0 0 0 0)
-	)
-	(junction
 		(at 93.98 99.06)
 		(diameter 0)
@@
 	(junction
 		(at 209.55 105.41)
-		(diameter 0)
-		(color 0 0 0 0)
-	)
-	(junction
-		(at 160.02 62.23)
 		(diameter 0)
 		(color 0 0 0 0)
@@
 	(wire
 		(pts
-			(xy 160.02 62.23) (xy 160.02 64.77)
+			(xy 160.02 44.45) (xy 160.02 64.77)
 		)
 		(stroke
@@
 	(wire
 		(pts
+			(xy 80.01 111.76) (xy 101.6 111.76)
+		)
+		(stroke
+			(width 0)
+			(type default)
+		)
+	)
+	(wire
+		(pts
 			(xy 209.55 128.27) (xy 209.55 130.81)
 		)
@@
 	(wire
 		(pts
-			(xy 97.79 116.84) (xy 101.6 116.84)
-		)
-		(stroke
-			(width 0)
-			(type default)
-		)
-	)
-	(wire
-		(pts
 			(xy 102.87 54.61) (xy 106.68 54.61)
 		)
@@
 	(wire
 		(pts
-			(xy 157.48 59.69) (xy 160.02 59.69)
-		)
-		(stroke
-			(width 0)
-			(type default)
-		)
-	)
-	(wire
-		(pts
 			(xy 158.75 168.91) (xy 158.75 175.26)
 		)
@@
 	(wire
 		(pts
-			(xy 160.02 59.69) (xy 160.02 62.23)
-		)
-		(stroke
-			(width 0)
-			(type default)
-		)
-	)
-	(wire
-		(pts
 			(xy 257.81 57.15) (xy 257.81 68.58)
 		)
@@
 	(wire
 		(pts
+			(xy 80.01 116.84) (xy 101.6 116.84)
+		)
+		(stroke
+			(width 0)
+			(type default)
+		)
+	)
+	(wire
+		(pts
 			(xy 260.35 52.07) (xy 278.13 52.07)
 		)
@@
 	(wire
 		(pts
-			(xy 93.98 111.76) (xy 93.98 104.14)
-		)
-		(stroke
-			(width 0)
-			(type default)
-		)
-	)
-	(wire
-		(pts
 			(xy 255.27 100.33) (xy 241.3 100.33)
 		)
@@
 	(wire
 		(pts
+			(xy 157.48 62.23) (xy 179.07 62.23)
+		)
+		(stroke
+			(width 0)
+			(type default)
+		)
+	)
+	(wire
+		(pts
 			(xy 133.35 146.05) (xy 133.35 154.94)
 		)
@@
 	(wire
 		(pts
-			(xy 93.98 111.76) (xy 101.6 111.76)
-		)
-		(stroke
-			(width 0)
-			(type default)
-		)
-	)
-	(wire
-		(pts
-			(xy 97.79 101.6) (xy 97.79 116.84)
-		)
-		(stroke
-			(width 0)
-			(type default)
-		)
-	)
-	(wire
-		(pts
 			(xy 31.75 144.78) (xy 31.75 152.4)
 		)
@@
 	(wire
 		(pts
-			(xy 157.48 62.23) (xy 160.02 62.23)
-		)
-		(stroke
-			(width 0)
-			(type default)
-		)
-	)
-	(wire
-		(pts
 			(xy 222.25 95.25) (xy 255.27 95.25)
 		)
@@
 	(wire
 		(pts
-			(xy 160.02 44.45) (xy 160.02 59.69)
-		)
-		(stroke
-			(width 0)
-			(type default)
-		)
-	)
-	(wire
-		(pts
 			(xy 149.86 154.94) (xy 158.75 154.94)
 		)
@@
 	(wire
 		(pts
+			(xy 157.48 59.69) (xy 179.07 59.69)
+		)
+		(stroke
+			(width 0)
+			(type default)
+		)
+	)
+	(wire
+		(pts
 			(xy 72.39 21.59) (xy 71.12 21.59)
 		)
@@
 	(wire
 		(pts
-			(xy 97.79 116.84) (xy 97.79 123.19)
+			(xy 97.79 101.6) (xy 97.79 123.19)
 		)
 		(stroke
@@
 			(width 0)
 			(type default)
+		)
+	)
+	(label "LCD_CS"
+		(at 179.07 59.69 180)
+		(effects
+			(font
+				(size 1.27 1.27)
+			)
+			(justify right bottom)
 		)
 	)
@@
 		)
 	)
+	(label "LCD_RESET"
+		(at 80.01 111.76 0)
+		(effects
+			(font
+				(size 1.27 1.27)
+			)
+			(justify left bottom)
+		)
+	)
 	(label "LCD_SCK"
 		(at 80.01 106.68 0)
@@
 		)
 	)
+	(label "LCD_RESET"
+		(at 179.07 62.23 180)
+		(effects
+			(font
+				(size 1.27 1.27)
+			)
+			(justify right bottom)
+		)
+	)
 	(label "UART1_TX"
 		(at 92.71 49.53 0)
@@
 		)
 	)
+	(label "LCD_CS"
+		(at 80.01 116.84 0)
+		(effects
+			(font
+				(size 1.27 1.27)
+			)
+			(justify left bottom)
+		)
+	)
