File: NitrogenGenerator.kicad_sch (KiCad schematic)
At the start: 27 parts, among them J1 Conn_ARM_SWD_TagConnect_TC203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, J2 Screw_Terminal_01x10, J3 ERM19264-4, J4 726386-2, J5 726386-2, J6 Conn_01x06_Pin, K1 AA28F-R1, K2 AA28F-R1, U1 STM32G030F6Px, U2 IRM-45-24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

Commit message: .
Parts:
- added C8, C9: 22nF, Capacitor_SMD:C_0603_1608Metric, symbol Device:C
Connections:
- net GND: now also C8.1, C9.1
- net at J2.10 (Pin_10), R4.2: now also C9.2
- net at J2.7 (Pin_7), R3.2: now also C8.2
Other:
- moved on the sheet: C5, C6, R3, R4, R5, R6

Commit message: .
Parts:
- added R7: 100, Resistor_SMD:R_0603_1608Metric, symbol Device:R
Connections:
- net +3.3V: no longer J3.2 (Pin_2)
- net +5V: now also R7.2
- new net: J3.2 (Pin_2), R7.1
Changed lines of the file:
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@@
 	)
 	(junction
-		(at 93.98 99.06)
-		(diameter 0)
-		(color 0 0 0 0)
-	)
-	(junction
 		(at 121.92 162.56)
 		(diameter 0)
@@
 	(wire
 		(pts
-			(xy 93.98 99.06) (xy 101.6 99.06)
+			(xy 233.68 113.03) (xy 233.68 120.65)
 		)
 		(stroke
@@
 	(wire
 		(pts
-			(xy 233.68 113.03) (xy 233.68 120.65)
+			(xy 80.01 92.71) (xy 80.01 99.06)
 		)
 		(stroke
@@
 	(wire
 		(pts
+			(xy 101.6 99.06) (xy 80.01 99.06)
+		)
+		(stroke
+			(width 0)
+			(type default)
+		)
+	)
+	(wire
+		(pts
 			(xy 241.3 107.95) (xy 241.3 100.33)
 		)
@@
 	(wire
 		(pts
-			(xy 93.98 93.98) (xy 93.98 99.06)
+			(xy 80.01 77.47) (xy 80.01 85.09)
 		)
 		(stroke
@@
 	(wire
 		(pts
-			(xy 93.98 99.06) (xy 93.98 104.14)
+			(xy 93.98 93.98) (xy 93.98 104.14)
 		)
 		(stroke
@@
 	)
 	(symbol
+		(lib_id "power:+5V")
+		(at 80.01 77.47 0)
+		(unit 1)
+		(exclude_from_sim no)
+		(in_bom yes)
+		(on_board yes)
+		(dnp no)
+		(fields_autoplaced yes)
+		(property "Reference" "#PWR035"
+			(at 80.01 81.28 0)
+			(effects
+				(font
+					(size 1.27 1.27)
+				)
+				(hide yes)
+			)
+		)
+		(property "Value" "+5V"
+			(at 80.01 72.39 0)
+			(effects
+				(font
+					(size 1.27 1.27)
+				)
+			)
+		)
+		(property "Footprint" ""
+			(at 80.01 77.47 0)
+			(effects
+				(font
+					(size 1.27 1.27)
+				)
+				(hide yes)
+			)
+		)
+		(property "Datasheet" ""
+			(at 80.01 77.47 0)
+			(effects
+				(font
+					(size 1.27 1.27)
+				)
+				(hide yes)
+			)
+		)
+		(property "Description" "Power symbol creates a global label with name \"+5V\""
+			(at 80.01 77.47 0)
+			(effects
+				(font
+					(size 1.27 1.27)
+				)
+				(hide yes)
+			)
+		)
+		(pin "1"
+		)
+		(instances
+			(project "NitrogenGenerator"
+				(path "/c5365556-9b4a-4e37-8bb8-20fd18113201"
+					(reference "#PWR035")
+					(unit 1)
+				)
+			)
+		)
+	)
+	(symbol
 		(lib_id "NitrogenGenerator:AA28F-R1")
 		(at 214.63 26.67 0)
@@
 					(unit 1)
 				)
+			)
+		)
+	)
+	(symbol
+		(lib_id "Device:R")
+		(at 80.01 88.9 180)
+		(unit 1)
+		(exclude_from_sim no)
+		(in_bom yes)
+		(on_board yes)
+		(dnp no)
+		(property "Reference" "R7"
+			(at 83.312 89.154 90)
+			(effects
+				(font
+					(size 1.27 1.27)
+				)
+			)
+		)
+		(property "Value" "100"
+			(at 85.852 89.154 90)
+			(effects
+				(font
+					(size 1.27 1.27)
+				)
+			)
+		)
+		(property "Footprint" "Resistor_SMD:R_0603_1608Metric"
+			(at 81.788 88.9 90)
+			(effects
+				(font
+					(size 1.27 1.27)
+				)
+				(hide yes)
+			)
+		)
+		(property "Datasheet" "~"
+			(at 80.01 88.9 0)
+			(effects
+				(font
+					(size 1.27 1.27)
+				)
+				(hide yes)
+			)
+		)
+		(property "Description" "Resistor"
+			(at 80.01 88.9 0)
+			(effects
+				(font
+					(size 1.27 1.27)
+				)
+				(hide yes)
+			)
+		)
+		(pin "2"
+		)
+		(pin "1"
+		)
+		(instances
+			(project "NitrogenGenerator"
+				(path "/c5365556-9b4a-4e37-8bb8-20fd18113201"
+					(reference "R7")
+					(unit 1)
+				)
